File: designs/ADC_Board_rev3/adc_cap.sch (EAGLE design)
At the start: 35 parts, among them Q1 BSS84, Q2 BSS84, Q3 BSS84, Q4 BSS84

Commit message: Update on adc rev 3
Parts:
- removed C7, C8, C9: (no value), rcl:C-USC0805
- removed R5, R7, R8: (no value), adafruit:R-US_R0805
- removed U$14: 2_X_8_CON, 11_pin_connecterp:2_X_8_CON
- added C14, C15, C16: (no value), rcl:C-USC1206K
- added R10, R11, R13: (no value), rcl:R-US_R1206W
- added U$2: 3020-16-0300-00, TIparts:3020-16-0300-00
- added U$5, U$9: 75869-103LF, TIparts:75869-103LF
- C1, C10, C11, C13, C2, C3, C4, C5, C6: device rcl:C-USC0805 -> rcl:C-USC1206K
- R1, R12, R2, R3, R4, R6, R9: device adafruit:R-US_R0805 -> rcl:R-US_R1206W
- U$7: value 2_X_8_CON -> 3020-16-0300-00; device 11_pin_connecterp:2_X_8_CON -> TIparts:3020-16-0300-00
Connections:
- removed net N$11: C1.1, R2.2, U$3.VDD
- new net N$37: U$7.1, U$8.CH0
- net GND: now also C13.1, C14.2, C15.2, C16.1, C3.1, C6.1, U$2.10, U$2.11, U$2.12, U$2.13, U$2.14, U$2.9, U$3.COM, U$4.COM, U$5.10, U$5.11, U$5.12, U$5.13, U$5.14, U$5.9, U$6.COM, U$8.COM, U$9.10, U$9.11, U$9.12, U$9.13, U$9.14, U$9.9; no longer C13.2, C3.2, C6.2, C7.2, C8.2, C9.2, U$14.10, U$14.11, U$14.12, U$14.13, U$14.14, U$14.9
- net N$1: now also U$2.1; no longer U$14.8
- net N$10: no longer R5.2
- net N$12: now also C13.2, R3.1; no longer C2.1
- net N$13: now also R13.2; no longer R3.2, R7.2, R8.1
- net N$14: now also C1.1, U$5.15, U$5.16; no longer C4.1
- net N$15: now also U$5.1
- net N$16: now also U$5.2
- net N$17: now also U$5.3
- net N$18: now also U$5.4
- net N$19: now also U$5.5
- net N$2: now also R12.2; no longer R1.2, R4.2, R5.1
- net N$20: now also U$5.6
- net N$21: now also U$5.7
- net N$22: now also U$5.8
- net N$23: no longer R4.1
- net N$24: no longer R8.2
- net N$25: now also C11.1, R11.2, R3.2, U$3.A1, U$3.VDD; no longer C5.1, R6.2, U$4.VDD
- net N$26: now also C3.2, R2.1; no longer C6.1
- net N$27: now also C4.1, U$9.15, U$9.16; no longer C7.1
- net N$28: now also U$9.1
- net N$29: now also U$9.2
- net N$3: now also U$2.2; no longer U$14.7
- net N$30: now also U$9.3
- net N$31: now also U$9.4
- net N$32: now also U$9.5
- net N$33: now also U$9.6
- net N$34: now also U$9.7
- net N$35: now also U$9.8
- net N$36: no longer R7.1
- net N$38: now also C2.1, R2.2, U$4.A0, U$4.VDD; no longer C8.1, U$6.VDD
- net N$39: now also C6.2, R1.1; no longer C9.1
- net N$4: now also U$2.3; no longer U$14.6
- net N$40: now also C14.1; no longer C10.1
- net N$41: now also U$7.2, U$8.CH1; no longer U$7.8, U$8.CH0
- net N$42: now also U$7.3, U$8.CH2; no longer U$7.7, U$8.CH1
- net N$43: now also U$7.4, U$8.CH3; no longer U$7.6, U$8.CH2
- net N$44: now also U$8.CH4; no longer U$8.CH3
- net N$45: now also U$7.6, U$8.CH5; no longer U$7.4, U$8.CH4
- net N$46: now also U$7.7, U$8.CH6; no longer U$7.3, U$8.CH5
- net N$47: now also U$7.8, U$8.CH7; no longer U$7.2, U$8.CH6
- net N$48: now also C5.1, R1.2, R10.2, U$6.A0, U$6.A1, U$6.VDD; no longer U$7.1, U$8.CH7
- net N$5: now also U$2.4; no longer U$14.5
- net N$51: now also C15.1, R4.2, R6.2; no longer C11.1, R12.2
- net N$52: now also C16.2, R4.1; no longer C13.1
- net N$6: now also U$2.5; no longer U$14.4
- net N$7: now also U$2.6; no longer U$14.3
- net N$76: now also C10.1, U$2.15, U$2.16; no longer C3.1, U$14.15, U$14.16
- net N$8: now also U$2.7; no longer U$14.2
- net N$9: now also U$2.8; no longer U$14.1
- net VCC: now also R10.1, R11.1, R13.1; no longer R1.1, R2.1, R3.1, U$3.A1, U$4.A0, U$6.A0, U$6.A1
Other:
- moved on the sheet: C1, C10, C11, C13, C2, C3, C4, C5, C6, R1, R12, R2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

Commit message: Done with ADC cap rev 3
Parts:
- added C17, C18, C7, C8, C9: (no value), rcl:C-USC1206K
- added J1, J2, J3, J4: 22-05-7028-02, con-molex:22-05-7028-02
- added LED1, LED2, LED3, LED4, LED5, LED6, LED7, LED8, LED9: (no value), led:LEDSML1206
- added R14, R15, R16, R17, R18, R19, R20, R21, R22, R23, R24, R25, R26, R27, R28, R29, R30, R31, R5, R7, R8: (no value), rcl:R-US_R1206W
- added U$10: CAS-220TB, TIparts:CAS-220TB
- added U$11: ISL23348_SD, TIparts:ISL23348_SD
- added U$12: MMPQ2907A, TIparts:MMPQ2907A
Connections:
- removed net N$76: C10.1, Q4.D, U$2.15, U$2.16
- new net GND4: R15.1
- new net N$11: U$1.I2C2_SDA, U$10.L4
- new net N$49: LED1.C, R5.2
- new net N$50: R27.1, U$11.RW1
- new net N$53: C1.1, LED2.A, Q1.D, U$5.15, U$5.16
- new net N$54: LED2.C, R7.2
- new net N$55: C10.1, LED3.A, Q4.D, U$2.15, U$2.16
- new net N$56: LED3.C, R8.2
- new net N$57: C14.1, LED4.A, Q3.D, U$7.15, U$7.16
- new net N$58: LED4.C, R14.2
- new net N$59: LED8.A, R17.1
- new net N$60: LED5.C, R15.2
- new net N$61: J4-1.S, R23.2, U$11.RL0
- new net N$62: J3-1.S, R26.2, U$11.RL1
- new net N$63: J2-1.S, R22.2, U$11.RL2
- new net N$64: J1-1.S, R21.2, U$11.RL3
- new net N$65: LED9.A, R16.1
- new net N$66: LED7.A, R18.1
- new net N$67: LED6.A, R20.1
- new net N$68: C17.2, R23.1, U$12.B4
- new net N$69: C18.2, R26.1, U$12.B3
- new net N$70: C9.2, R22.1, U$12.B1
- new net N$71: C8.2, R21.1, U$12.B2
- new net N$72: R16.2, R31.2, U$12.C1, U$12.C1'
- new net N$73: R17.2, R30.2, U$12.C2, U$12.C2'
- new net N$74: R18.2, R29.2, U$12.C3, U$12.C3'
- new net N$75: R20.2, R28.2, U$12.C4, U$12.C4'
- net GND: now also C17.1, C18.1, C7.2, C8.1, C9.1, J1-2.S, J2-2.S, J3-2.S, J4-2.S, LED6.C, LED7.C, LED8.C, LED9.C, R14.1, R28.1, R29.1, R30.1, R31.1, R5.1, R7.1, R8.1, U$11.A0, U$11.A1, U$11.A2, U$11.GND
- net N$10: now also U$1.I2C1_SDA, U$10.L3; no longer U$1.I2C2_SDA
- net N$13: now also U$10.C1, U$11.SCL
- net N$14: now also R19.1, U$11.RW3; no longer C1.1, Q1.D, U$5.15, U$5.16
- net N$2: now also U$10.C2, U$11.SDA
- net N$23: now also U$1.I2C1_SCL, U$10.L1; no longer U$1.I2C1_SDA
- net N$24: now also U$10.L2
- net N$27: now also LED1.A
- net N$36: now also R24.1, U$11.RW2; no longer U$1.I2C1_SCL
- net N$40: now also R25.1, U$11.RW0; no longer C14.1, Q3.D, U$7.15, U$7.16
- net VCC: now also C7.1, LED5.A, R19.2, R24.2, R25.2, R27.2, U$11.VCC, U$11.VLOGIC, U$12.E1, U$12.E2, U$12.E3, U$12.E4

Commit message: done with adc rev3
Parts:
- added C19: (no value), rcl:C-USC1206K
- added J5: 22-05-7058-05, con-molex:22-05-7058-05
- renumbered LED1 to LEFT, LED2 to RIGHT, LED3 to BACK, LED4 to FRONT, LED5 to POWER
Connections:
- removed net N$72: R16.2, R31.2, U$12.C1, U$12.C1'
- removed net N$74: R18.2, R29.2, U$12.C3, U$12.C3'
- removed net N$75: R20.2, R28.2, U$12.C4, U$12.C4'
- new net N$77: R17.2, R30.2, U$1.UART4_TXD, U$12.C2, U$12.C2'
- new net N$78: R20.2, R28.2, U$1.UART4_RXD, U$12.C4, U$12.C4'
- new net N$79: R18.2, R29.2, U$1.GPIO1_28, U$12.C3, U$12.C3'
- new net N$80: R16.2, R31.2, U$1.GPIO1_16, U$12.C1, U$12.C1'
- net GND: now also C19.2, J5-1.S
- net N$13: now also J5-5.S
- net N$2: now also J5-4.S
- net N$73: now also J5-3.S, U$1.GPIO1_7; no longer R17.2, R30.2, U$12.C2, U$12.C2'
- net VCC: now also C19.1, J5-2.S
